Commit message: spawn box model

File: urdf/cs_test_box2.xacro (robot description, xacro)
@@ -3,11 +3,11 @@
 <link name="cs_test_box1">
     <visual>
-        <origin xyz="0 0 2" rpy="0 0 0"/>
+        <origin xyz="3 3 2" rpy="0 0 0"/>
       <geometry>
         <mesh filename="package://cs_test/models/box.dae" scale="0.5 0.5 0.5"/>
       </geometry>
     </visual>
-    <collision name="box1">
-        <origin xyz="0 0 2" rpy="0 0 0"/>
+    <collision name="box2">
+        <origin xyz="3 3 2" rpy="0 0 0"/>
       <geometry>
         <mesh filename="package://cs_test/models/box.dae" scale="0.5 0.5 0.5"/>
@@ -15,10 +15,10 @@
     </collision>
     <inertial>
-        <origin xyz="0 0 2" rpy="0 0 0"/>
+        <origin xyz="3 3 2" rpy="0 0 0"/>
         <mass value="1"/>
         <inertia ixx="0.083"  ixy="0"  ixz="0" iyy="0.083" iyz="0" izz="0.083"/>
     </inertial>
 </link>
-<gazebo reference="cs_test_box1">
+<gazebo reference="cs_test_box2">
     <mu1 value="200" />
     <mu2 value="100" />
