Commit message: spawn two base

File: urdf/cs_test.xacro (robot description, xacro)
@@ -6,7 +6,7 @@
       <origin xyz="0 0 0" rpy="0 0 0"/>
       <parent link="world"/>
-      <child link="base"/>
+      <child link="base1"/>
     </joint>
-<link name="base">
+<link name="base1">
     <visual>
         <origin xyz="0 0 0.6" rpy="0 0 0"/>
@@ -15,5 +15,5 @@
       </geometry>
     </visual>
-    <collision name="base">
+    <collision name="base1">
         <origin xyz="0 0 0.6" rpy="0 0 0"/>
       <geometry>
@@ -27,5 +27,30 @@
     </inertial>
 </link>
-<gazebo reference="base">
+    <joint name="joint2" type="fixed">
+      <axis xyz="0 0 0"/>
+      <origin xyz="0 0 0" rpy="0 0 0"/>
+      <parent link="world"/>
+      <child link="base2"/>
+    </joint>
+<link name="base2">
+    <visual>
+        <origin xyz="3 3 0.1" rpy="0 0 0"/>
+      <geometry>
+        <mesh filename="package://cs_test/models/box.dae" scale="1 1 0.01"/>
+      </geometry>
+    </visual>
+    <collision name="base2">
+        <origin xyz="3 3 0.1" rpy="0 0 0"/>
+      <geometry>
+        <mesh filename="package://cs_test/models/box.dae" scale="1 1 0.01"/>
+      </geometry>
+    </collision>
+    <inertial>
+        <origin xyz="3 3 0.1" rpy="0 0 0"/>
+        <mass value="1"/>
+        <inertia ixx="0.083"  ixy="0"  ixz="0" iyy="0.083" iyz="0" izz="0.083"/>
+    </inertial>
+</link>
+<gazebo reference="base1">
     <mu1 value="200" />
     <mu2 value="100" />
@@ -35,5 +60,5 @@
     <update_rate>100.0</update_rate>
     <contact>
-      <collision>base_collision</collision>
+      <collision>base1_collision</collision>
     </contact>
     <plugin name="cs_test" filename="libcs_test.so">
@@ -43,3 +68,19 @@
    </sensor>
 </gazebo>
+<gazebo reference="base2">
+    <mu1 value="200" />
+    <mu2 value="100" />
+    <selfCollide>true</selfCollide>
+    <sensor name="contact_sensor" type="contact">
+    <always_on>true</always_on>
+    <update_rate>100.0</update_rate>
+    <contact>
+      <collision>base2_collision</collision>
+    </contact>
+    <plugin name="cs_test" filename="libcs_test.so">
+      <bumperTopicName>state2</bumperTopicName>
+      <frameName>world</frameName>
+    </plugin>
+   </sensor>
+</gazebo>
 </robot>

Commit message: change mass value

File: urdf/cs_test.xacro (robot description, xacro)
@@ -64,5 +64,5 @@
     <plugin name="cs_test" filename="libcs_test.so">
       <bumperTopicName>state1</bumperTopicName>
-      <frameName>world</frameName>
+      <frameName>base1</frameName>
     </plugin>
    </sensor>
@@ -80,5 +80,5 @@
     <plugin name="cs_test" filename="libcs_test.so">
       <bumperTopicName>state2</bumperTopicName>
-      <frameName>world</frameName>
+      <frameName>base2</frameName>
     </plugin>
    </sensor>

File: urdf/cs_test_box.xacro (robot description, xacro)
@@ -16,5 +16,5 @@
     <inertial>
         <origin xyz="0 0 2" rpy="0 0 0"/>
-        <mass value="1"/>
+        <mass value="0.3"/>
         <inertia ixx="0.083"  ixy="0"  ixz="0" iyy="0.083" iyz="0" izz="0.083"/>
     </inertial>

Commit message: rescale size and change position for experiment

File: urdf/cs_test.xacro (robot description, xacro)
@@ -12,5 +12,5 @@
         <origin xyz="0 0 0.6" rpy="0 0 0"/>
       <geometry>
-        <mesh filename="package://cs_test/models/box.dae"/>
+        <mesh filename="package://cs_test/models/box.dae" scale="4 4 1"/>
       </geometry>
     </visual>
@@ -18,5 +18,5 @@
         <origin xyz="0 0 0.6" rpy="0 0 0"/>
       <geometry>
-        <mesh filename="package://cs_test/models/box.dae"/>
+        <mesh filename="package://cs_test/models/box.dae" scale="4 4 1"/>
       </geometry>
     </collision>

File: urdf/cs_test_box.xacro (robot description, xacro)
@@ -3,17 +3,17 @@
 <link name="cs_test_box1">
     <visual>
-        <origin xyz="0 0 2" rpy="0 0 0"/>
+        <origin xyz="0 -0.6 1.5" rpy="0 0 0"/>
       <geometry>
-        <mesh filename="package://cs_test/models/box.dae" scale="0.5 0.5 0.5"/>
+        <mesh filename="package://cs_test/models/box.dae" scale="0.1 0.1 0.1"/>
       </geometry>
     </visual>
     <collision name="box1">
-        <origin xyz="0 0 2" rpy="0 0 0"/>
+        <origin xyz="0 -0.6 1.5" rpy="0 0 0"/>
       <geometry>
-        <mesh filename="package://cs_test/models/box.dae" scale="0.5 0.5 0.5"/>
+        <mesh filename="package://cs_test/models/box.dae" scale="0.1 0.1 0.1"/>
       </geometry>
     </collision>
     <inertial>
-        <origin xyz="0 0 2" rpy="0 0 0"/>
+        <origin xyz="0 -0.6 1.5" rpy="0 0 0"/>
         <mass value="0.3"/>
         <inertia ixx="0.083"  ixy="0"  ixz="0" iyy="0.083" iyz="0" izz="0.083"/>

File: urdf/cs_test_box2.xacro (robot description, xacro)
@@ -5,5 +5,5 @@
         <origin xyz="3 3 2" rpy="0 0 0"/>
       <geometry>
-        <mesh filename="package://cs_test/models/box.dae" scale="0.5 0.5 0.5"/>
+        <mesh filename="package://cs_test/models/box.dae" scale="0.1 0.1 0.1"/>
       </geometry>
     </visual>
@@ -11,5 +11,5 @@
         <origin xyz="3 3 2" rpy="0 0 0"/>
       <geometry>
-        <mesh filename="package://cs_test/models/box.dae" scale="0.5 0.5 0.5"/>
+        <mesh filename="package://cs_test/models/box.dae" scale="0.1 0.1 0.1"/>
       </geometry>
     </collision>
